File: hardware/navigator.kicad_sch (KiCad schematic)
At the start: 41 parts, among them J1 BLDC-1, J10 GPIO, J2 BLDC-1, J3 BLDC-1, J4 BLDC-1, J5 BLDC-1, J6 BLDC-1, J7 Conn_01x02_Pin, J8 USB_C_Receptacle_USB2.0_16P, J9 Conn_01x04_Pin, SW1 SW_SPST, SW2 SW_SPST, U1 AP2112K-3.3, U2 LM2576-5.0, U3 ESP32-S3-MINI-1U, U4 INA226

Commit message: feat: update navigator hardware to revision 002
Parts:
- removed C1: 0.1uF, Capacitor_SMD:C_0805_2012Metric, symbol Device:C
- removed C2: 330uF, Capacitor_SMD:C_Elec_10x10.2, symbol Device:C_Polarized
- removed D1: Schottky, Diode_SMD:D_SMB, symbol Device:D_Schottky
- removed L1: 100uH, Inductor_SMD:L_Vishay_IHLP-6767, symbol Device:L
- removed U2: LM2576-5.0, Package_TO_SOT_SMD:TO-263-5_TabPin3, symbol Regulator_Switching:LM2576HVS-5
- added C1: 100uF, Capacitor_SMD:CP_Elec_8x10.5, symbol Device:C_Polarized
- added C10, C8, C9: 0.1uF, Capacitor_SMD:C_0805_2012Metric, symbol Device:C
- added C2: 10uF, Capacitor_SMD:C_1210_3225Metric, symbol Device:C
- added R14, R15, R16, R9: 10k, Resistor_SMD:R_0805_2012Metric, symbol Device:R
- added R7: 100k, Resistor_SMD:R_0805_2012Metric, symbol Device:R
- added R8: 14k3, Resistor_SMD:R_0805_2012Metric, symbol Device:R
- added U2: MPM3550EGLE, Package_LGA:MPS_LGA-18-10EP_12x12mm_P3.3mm, symbol Regulator_Switching:MPM3550EGLE
- added U3: BNO086, BNO086:BNO086, symbol BNO086:BNO086
- C3, C6: DigiKey_PN 587-1299-1-ND -> 1276-2872-1-ND
- C5: value 1000uF -> 47uF; footprint Capacitor_SMD:CP_Elec_10x10.5 -> Capacitor_SMD:C_1210_3225Metric; DigiKey_PN P122428CT-ND -> GRM32ER61C476ME15L
- C7: footprint Capacitor_SMD:C_0603_1608Metric -> Capacitor_SMD:C_0805_2012Metric; DigiKey_PN 399-C0603C104K5RACTUCT-ND -> 1276-1003-1-ND
- J7: footprint Connector_JST:JST_VH_S2P-VH_1x02_P3.96mm_Horizontal -> 282837-2:282837-2; DigiKey_PN 455-S2P-VH-ND -> A113320-ND
- renumbered C10 to C11, C8 to C12, C9 to C13, D2 to D1, D3 to D2, R9 to R10, R10 to R11, R7 to R12, R8 to R13, R11 to R17, SW2 to SW1, SW1 to SW2, U3 to U4, U4 to U5
Connections:
- net +3V3: now also C10.1, C8.1, R14.2, R15.1, R16.2, R9.1, U3.10 (CLKSEL0), U3.28 (VDDIO), U3.3 (VDD)
- net +BATT: now also C1.1, C2.2, U2.8 (VIN)
- net BUCK_5V: now also U2.5 (VOUT)
- net GND: now also J1.3 (Pin_3), R1.2, C1.2, C10.2, C2.1, C8.2, C9.2, R7.1, R8.2, U2.10 (GND), U2.11 (GND), U2.12 (GND), U2.13 (GND), U2.14 (GND), U2.15 (GND), U2.16 (GND), U2.17 (GND), U2.18 (GND), U2.6 (GND), U2.7 (GND), U2.9 (GND), U3.17 (SA0/H_MOSI), U3.2 (GND), U3.25 (GNDIO), U3.26 (XOUT32/CLKSEL1), U3.5 (PS1), U3.6 (PS0/WAKE)
- net GPIO14/TXD0: now also U4.22 (IO18); no longer U4.40 (RXD0)
- net GPIO15/RXD0: now also U4.21 (IO17); no longer U4.39 (TXD0)
- net I2C_SCL: now also U3.19 (H_SCL/SCK/RX)
- net I2C_SDA: now also U3.20 (H_SDA/H_MISO/TX)
- new net: R14.1, U3.11 (~{RST})
- new net: C9.1, U3.9 (CAP)
- new net: R7.2, U2.2 (RFREQ)
- new net: R8.1, U2.4 (FB)
- new net: R16.1, U3.15 (ENV_SCL)
- new net: U3.1 (RESV_NC), U3.12 (RESV_NC), U3.13 (RESV_NC), U3.21 (RESV_NC), U3.22 (RESV_NC), U3.23 (RESV_NC), U3.24 (RESV_NC), U3.7 (RESV_NC), U3.8 (RESV_NC)
- new net: R15.2, U3.16 (ENV_SDA)
- new net: R9.2, U3.4 (~{BOOT})
- no-connect marks 63 -> 68
Other:
- note removed: "C2, C5 must be aluminum electrolytic and support 35V Ensure D1 is Schottky and supports 3A"
- moved on the sheet: C12, C13, C3, C4, C6, C7, D1, D2, J9, R12, R13, R17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
